File: simplevideo/simplevideo.kicad_pcb (KiCad board)
At the start: 2 copper layers, 28 parts, among them Q2 2N3904, U1 4040, U10 CD74HC40103, U11 CD74HC40103, U12 CD74HC40103, U13 74LS74, U14 CD74HC40103, U15 CD74HC40103, U16 CD74HC40103, U17 74LS74, U18 74HCT00, U2 CD74HC40103, U3 CD74HC40103, U4 4040, U5 4040, U6 74HC74, U7 CD74HC40103, U8 CD74HC40103, X1 CXO_DIP8

Commit message: Include 6502, ROM, etc in circuit, all laid out together
Parts:
- added J1: Conn_01x02, Connector_PinHeader_2.54mm:PinHeader_1x02_P2.54mm_Vertical, F.Cu at (185.4, 114.3)
- added J2: Conn_01x08, Connector_PinHeader_2.54mm:PinHeader_1x08_P2.54mm_Vertical, F.Cu at (99.1, 203.2)
- added J3: Conn_01x08, Connector_PinHeader_2.54mm:PinHeader_1x08_P2.54mm_Vertical, F.Cu at (30.5, 231.1)
- added J4: Conn_01x08, Connector_PinHeader_2.54mm:PinHeader_1x08_P2.54mm_Vertical, F.Cu at (55.9, 231.1)
- added R2: 1K, Resistor_THT:R_Axial_DIN0207_L6.3mm_D2.5mm_P7.62mm_Horizontal, F.Cu at (78.7, 147.3)
- added U19: 74LS00, Package_DIP:DIP-14_W7.62mm, F.Cu at (78.7, 109.2)
- added U20: 74HC74, Package_DIP:DIP-14_W7.62mm, F.Cu at (119.4, 109.2)
- added U21: 74LS245, Package_DIP:DIP-20_W7.62mm, F.Cu at (142.2, 165.1)
- added U22: 74LS32, Package_DIP:DIP-14_W7.62mm, F.Cu at (139.7, 109.2)
- added U23: 74LS245, Package_DIP:DIP-20_W7.62mm, F.Cu at (27.9, 221.0)
- added U24: 74LS245, Package_DIP:DIP-20_W7.62mm, F.Cu at (30.5, 165.1)
- added U25: 74LS166, Package_DIP:DIP-16_W7.62mm, F.Cu at (121.9, 165.1)
- added U26: 62256, Package_DIP:DIP-28_W15.24mm, F.Cu at (83.8, 167.6)
- added U27: 28C256, Package_DIP:DIP-28_W15.24mm, F.Cu at (134.6, 223.5)
- added U28: 74LS245, Package_DIP:DIP-20_W7.62mm, F.Cu at (53.3, 221.0)
- added U29: 74LS245, Package_DIP:DIP-20_W7.62mm, F.Cu at (55.9, 165.1)
- added U30: 74HC74, Package_DIP:DIP-14_W7.62mm, F.Cu at (40.6, 53.3)
- added U31: 74HC74, Package_DIP:DIP-14_W7.62mm, F.Cu at (61.0, 53.3)
- added U32: 74LS138, Package_DIP:DIP-16_W7.62mm, F.Cu at (167.6, 165.1)
- added U9: 74HC74, Package_DIP:DIP-14_W7.62mm, F.Cu at (99.1, 109.2)
- U18: value 74HCT00 -> WD65C02_; footprint Package_DIP:DIP-14_W7.62mm -> Package_DIP:DIP-40_W15.24mm
- U2: value CD74HC40103 -> 74LS08; footprint Package_DIP:DIP-16_W7.62mm -> Package_DIP:DIP-14_W7.62mm
- moved U18 232.3 mm to (81.3, 223.5)
- moved R8 179.6 mm to (185.4, 109.2), turned to 90 degrees
- moved R10 176.9 mm to (185.4, 83.8)
- moved Q2 175.0 mm to (184.2, 99.1), turned to 180 degrees
- moved R9 173.0 mm to (182.9, 83.8)
- moved D1 169.9 mm to (168.9, 96.5)
- moved R4 166.6 mm to (180.3, 109.2), turned to 90 degrees
- moved R7 164.2 mm to (182.9, 94.0)
- moved U2 131.8 mm to (160.0, 109.2)
- moved U1 99.8 mm to (-27.9, 83.8)
- moved U6 69.1 mm to (43.2, -2.54)
- moved U3 20.3 mm to (81.3, 53.3)
- moved U4 7.62 mm to (55.9, 109.2)
- moved U5 5.08 mm to (33.0, 109.2)
Connections:
- net Col0 renamed VCOL0
- net Col1 renamed VCOL1
- net Col10 renamed VCOL10
- net Col11 renamed VCOL11
- net Col2 renamed VCOL2
- net Col9 renamed VCOL9
- net Row10 renamed VROW10
- net Row11 renamed VROW11
- net Row9 renamed VROW9
- U15 pad 2: Net-(U15-Pad2) -> ~HOn
- U17 pad 5: Net-(U15-Pad2) -> ~HOn
- U18 pad 1: HOn -> Net-(U18-Pad1)
- U18 pad 10: Net-(U18-Pad10) -> A1
- U18 pad 11: Net-(U18-Pad10) -> A2
- U18 pad 12: ~HSync -> A3
- U18 pad 13: ~VSync -> A4
- U18 pad 14: (no net) -> A5
- U18 pad 2: HOn -> VCC
- U18 pad 4: Net-(U18-Pad3) -> VCC
- U18 pad 5: Net-(U18-Pad3) -> Net-(U18-Pad5)
- U18 pad 6: Net-(R7-Pad2) -> VCC
- U18 pad 7: (no net) -> Net-(U18-Pad7)
- U18 pad 8: Net-(D1-Pad1) -> VCC
- U18 pad 9: Net-(U18-Pad10) -> A0
- U2 pad 1: 16MHz -> ~CPU_PHI_R
- U2 pad 10: GND -> LUM
- U2 pad 11: GND -> Net-(D1-Pad1)
- U2 pad 12: GND -> ~HSync
- U2 pad 13: GND -> ~VSync
- U2 pad 14: 4MHz -> (no net)
- U2 pad 2: VCC -> /Memory Controller/~GPUBUS
- U2 pad 3: GND -> Net-(U2-Pad3)
- U2 pad 4: VCC -> (no net)
- U2 pad 5: VCC -> (no net)
- U2 pad 6: GND -> (no net)
- U2 pad 7: GND -> (no net)
- U2 pad 8: GND -> Net-(R7-Pad2)
- U2 pad 9: VCC -> HOn
- U3 pad 13: VCC -> GND
- U4 pad 12: Row8 -> VROW8
- U4 pad 13: Row7 -> VROW7
- U4 pad 2: Row5 -> VROW5
- U4 pad 3: Row4 -> VROW4
- U4 pad 4: Row6 -> VROW6
- U4 pad 5: Row3 -> VROW3
- U4 pad 6: Row2 -> VROW2
- U4 pad 7: Row1 -> VROW1
- U4 pad 9: Row0 -> VROW0
- U5 pad 12: Col8 -> VCOL8
- U5 pad 13: Col7 -> VCOL7
- U5 pad 2: Col5 -> VCOL5
- U5 pad 3: Col4 -> VCOL4
- U5 pad 4: Col6 -> VCOL6
- U5 pad 5: Col3 -> VCOL3
- U6 pad 1: (no net) -> Net-(U6-Pad1)
- U6 pad 11: HalfRowClk -> ~2MHz
- U6 pad 12: RowClk -> ~RowClk
- U6 pad 2: (no net) -> ~RowClk
- U6 pad 3: (no net) -> HalfRowClk
- U6 pad 4: (no net) -> VCC
- U6 pad 5: (no net) -> RowClk
- U6 pad 6: (no net) -> ~RowClk
- U6 pad 8: RowClk -> Net-(U6-Pad8)
- U6 pad 9: Net-(U6-Pad9) -> Net-(U6-Pad1)
- X1 pad 5: 16MHz -> Net-(U30-Pad3)
Routing:
- net VCC: track 2639.6 -> 3077.2 mm, vias 170 -> 172
- net GND: track 2979.4 -> 3371.8 mm, vias 199 -> 190
- net (no net): track 40.6 -> 162.6 mm, vias 0 -> 1
- net 4MHz: track 170.2 -> 114.3 mm, vias 8 -> 5
- net RowClk: track 127.0 -> 83.8 mm, vias 8 -> 5
- net ~RowClk: track 0.00 -> 40.6 mm, vias 0 -> 2
- net Net-(U18-Pad3): track 35.6 -> 0.00 mm, vias 4 -> 0
- net Net-(U18-Pad10): track 35.6 -> 0.00 mm, vias 4 -> 0
- net Net-(U15-Pad2): track 33.0 -> 0.00 mm, vias 2 -> 0
- net 8MHz: track 0.00 -> 30.5 mm
- net Net-(U6-Pad1): track 0.00 -> 20.3 mm
- net Net-(U30-Pad3): track 0.00 -> 20.3 mm
- net 16MHz: track 20.3 -> 0.00 mm
- net ~VSync: track 50.8 -> 40.6 mm
- net ~HSync: track 50.8 -> 40.6 mm
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
Commit message: New address decoding scheme and complete breadboard layout, should be ready to build
Parts:
- removed U1: 4040, Package_DIP:DIP-16_W7.62mm
- added C1: 1u, Capacitor_THT:CP_Radial_D5.0mm_P2.50mm, F.Cu at (248.9, 30.5)
- added Q1: 2N3906, Package_TO_SOT_THT:TO-92_Inline, F.Cu at (248.9, 25.4)
- added Q3: 2N3904, Package_TO_SOT_THT:TO-92_Inline, F.Cu at (254.0, 30.5)
- added R3: 10K, Resistor_THT:R_Axial_DIN0207_L6.3mm_D2.5mm_P7.62mm_Horizontal, F.Cu at (236.2, 26.7)
- added R5: 100K, Resistor_THT:R_Axial_DIN0207_L6.3mm_D2.5mm_P7.62mm_Horizontal, F.Cu at (236.2, 29.2)
- added R6: 1K, Resistor_THT:R_Axial_DIN0207_L6.3mm_D2.5mm_P7.62mm_Horizontal, F.Cu at (246.4, 31.8)
- added SW1: SW_Push, Button_Switch_THT:SW_PUSH_6mm, F.Cu at (262.9, 34.3)
- moved J3 249.3 mm to (274.3, 179.1), turned to 180 degrees
- moved U23 239.5 mm to (264.2, 181.6), turned to 180 degrees
- moved J4 231.8 mm to (274.3, 153.7), turned to 180 degrees
- moved U28 220.5 mm to (264.2, 156.2), turned to 180 degrees
- moved U18 208.5 mm to (266.7, 128.3), turned to 180 degrees
- moved U27 198.8 mm to (266.7, 74.9), turned to 180 degrees
- moved U24 178.3 mm to (208.3, 179.1), turned to 180 degrees
- moved J2 174.1 mm to (246.4, 110.5), turned to 180 degrees
- moved R1 169.4 mm to (22.9, 143.5), turned to 180 degrees
- moved U6 168.9 mm to (40.6, 166.4), turned to 180 degrees
- moved D3 161.9 mm to (25.4, 137.2), turned to 90 degrees
- moved D2 160.2 mm to (30.5, 143.5), turned to 160 degrees
- moved U29 152.8 mm to (208.3, 153.7), turned to 180 degrees
- moved U7 150.3 mm to (40.6, 146.1), turned to 180 degrees
- moved X1 145.5 mm to (96.5, 181.6), turned to 90 degrees
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Connections:
- net CS0 renamed ~IOCS0
- net CS1 renamed ~IOCS1
- net CS2 renamed ~IOCS2
- net CS3 renamed ~IOCS3
- net CS4 renamed ~IOCS4
- net CS5 renamed ~IOCS5
- net CS6 renamed ~IOCS6
- R7 pad 2: Net-(R7-Pad2) -> LUM
- U15 pad 15: ~HSync -> ~RowClk
- U18 pad 40: VCC -> ~CPU_RESET
- U19 pad 10: 2MHz -> Net-(U19-Pad10)
- U19 pad 12: ~RowClk -> Net-(U19-Pad12)
- U19 pad 13: 1MHz -> Net-(U19-Pad13)
- U19 pad 8: Net-(U19-Pad8) -> ~ROMCS
- U19 pad 9: 1MHz -> A15
- U2 pad 10: LUM -> ~VSync
- U2 pad 11: Net-(D1-Pad1) -> Net-(U2-Pad11)
- U2 pad 12: ~HSync -> ~RowClk
- U2 pad 13: ~VSync -> 1MHz
- U2 pad 4: (no net) -> 1MHz
- U2 pad 5: (no net) -> 2MHz
- U2 pad 6: (no net) -> Net-(U2-Pad6)
- U2 pad 8: Net-(R7-Pad2) -> Net-(D1-Pad1)
- U2 pad 9: HOn -> ~HSync
- U22 pad 1: ~CPU_PHI_R -> ~CPU_PHI_W
- U22 pad 10: (no net) -> Net-(U22-Pad10)
- U22 pad 11: (no net) -> Net-(U22-Pad10)
- U22 pad 12: (no net) -> A13
- U22 pad 13: (no net) -> A12
- U22 pad 2: /Memory Controller/IA15 -> /Memory Controller/~AllowWrite
- U22 pad 3: Net-(U21-Pad1) -> Net-(U22-Pad3)
- U22 pad 4: ~CPU_PHI_W -> ~CPU_PHI_R
- U22 pad 5: /Memory Controller/~AllowWrite -> /Memory Controller/IA15
- U22 pad 6: Net-(U22-Pad6) -> Net-(U21-Pad1)
- U22 pad 8: (no net) -> Net-(U19-Pad10)
- U22 pad 9: (no net) -> A14
- U25 pad 9: VCC -> HOn
- U26 pad 27: Net-(U22-Pad6) -> Net-(U22-Pad3)
- U27 pad 20: CS7 -> ~ROMCS
- U30 pad 11: 8MHz -> Net-(U30-Pad11)
- U30 pad 12: 4MHz -> 8MHz
- U30 pad 2: 8MHz -> 4MHz
- U30 pad 3: Net-(U30-Pad3) -> 8MHz
- U30 pad 6: 8MHz -> 4MHz
- U30 pad 8: 4MHz -> 8MHz
- U31 pad 11: 2MHz -> Net-(U30-Pad5)
- U31 pad 12: Net-(U19-Pad11) -> 2MHz
- U31 pad 2: 2MHz -> Net-(U2-Pad11)
- U31 pad 3: Net-(U30-Pad9) -> 2MHz
- U31 pad 5: ~2MHz -> Net-(U31-Pad5)
- U31 pad 6: 2MHz -> 1MHz
- U31 pad 8: Net-(U31-Pad8) -> 2MHz
- U31 pad 9: 1MHz -> ~2MHz
- U32 pad 1: A12 -> A9
- U32 pad 2: A13 -> A10
- U32 pad 3: A14 -> A11
- U32 pad 5: GND -> Net-(U19-Pad10)
- U32 pad 7: CS7 -> ~IOCS7
- U9 pad 2: Net-(U19-Pad8) -> Net-(U2-Pad6)
- U9 pad 5: /Memory Controller/~AllowWrite -> Net-(U9-Pad5)
- U9 pad 6: Net-(U9-Pad6) -> /Memory Controller/~AllowWrite
- X1 pad 5: Net-(U30-Pad3) -> Net-(U30-Pad11)
Routing:
- net VCC: track 3077.2 -> 3731.3 mm, vias 172 -> 223
- net /Memory Controller/~GPUBUS: track 0.00 -> 288.3 mm, vias 0 -> 10
- net ~RowClk: track 40.6 -> 327.1 mm, vias 2 -> 8
- net GND: track 3371.8 -> 3656.4 mm, vias 190 -> 210
- net 4MHz: track 114.3 -> 362.3 mm, vias 5 -> 18
- net 1MHz: track 0.00 -> 190.1 mm, vias 0 -> 8
- net ~VSync: track 40.6 -> 205.2 mm, vias 2 -> 6
- net (no net): track 162.6 -> 0.00 mm, vias 1 -> 0
- net /Memory Controller/IA15: track 0.00 -> 158.8 mm, vias 0 -> 4
- net ~CPU_PHI_R: track 0.00 -> 142.9 mm, vias 0 -> 7
- net RowClk: track 83.8 -> 218.0 mm, vias 5 -> 8
- net ~HOn: track 33.0 -> 164.4 mm, vias 2 -> 6
- net ~CPU_RESET: track 0.00 -> 121.7 mm, vias 0 -> 4
- net ~2MHz: track 10.2 -> 121.0 mm, vias 0 -> 3
- net Net-(D1-Pad1): track 6.35 -> 115.4 mm, vias 1 -> 2
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Other:
- board outline added: 276.9 x 172.7 mm

Commit message: Fixed various issues discovered during building and testing
Parts:
- removed Q2: 2N3904, Package_TO_SOT_THT:TO-92_Inline
- added C10: 220u, Capacitor_THT:CP_Radial_D5.0mm_P2.50mm, F.Cu at (236.2, 128.3)
- added C11: 220u, Capacitor_THT:CP_Radial_D5.0mm_P2.50mm, F.Cu at (281.9, 149.9)
- added C2: 220u, Capacitor_THT:CP_Radial_D5.0mm_P2.50mm, F.Cu at (12.7, 151.1)
- added C3: 220u, Capacitor_THT:CP_Radial_D5.0mm_P2.50mm, F.Cu at (58.4, 153.7)
- added C4: 220u, Capacitor_THT:CP_Radial_D5.0mm_P2.50mm, F.Cu at (68.6, 151.1)
- added C5: 220u, Capacitor_THT:CP_Radial_D5.0mm_P2.50mm, F.Cu at (114.3, 154.9)
- added C6: 220u, Capacitor_THT:CP_Radial_D5.0mm_P2.50mm, F.Cu at (124.5, 149.9)
- added C7: 220u, Capacitor_THT:CP_Radial_D5.0mm_P2.50mm, F.Cu at (170.2, 132.1)
- added C8: 220u, Capacitor_THT:CP_Radial_D5.0mm_P2.50mm, F.Cu at (180.3, 118.1)
- added C9: 220u, Capacitor_THT:CP_Radial_D5.0mm_P2.50mm, F.Cu at (226.1, 124.5)
- added D4: 1N4148, Diode_THT:D_DO-34_SOD68_P7.62mm_Horizontal, F.Cu at (139.7, 34.3)
- added R11: 100K, Resistor_THT:R_Axial_DIN0207_L6.3mm_D2.5mm_P7.62mm_Horizontal, F.Cu at (274.3, 125.7)
- D1, D2, D3: value 1N4007 -> 1N4148
- R10: value 40 -> 47
- R4: value 38K -> 330
- R7: value 22K -> 200
- R8: value 40 -> 20
- R9: value 22K -> 2K2
- moved R10 29.7 mm to (154.9, 34.3), turned to 90 degrees
- moved R4 27.9 mm to (124.5, 29.2), turned to 0 degrees
- moved R7 12.7 mm to (144.8, 29.2), turned to 0 degrees
- moved J1 10.5 mm to (160.0, 34.3), turned to 180 degrees
- moved U18 2.54 mm to (269.2, 128.3)
- moved U26 2.54 mm to (213.4, 125.7)
- moved U27 2.54 mm to (269.2, 74.9)
- moved R9 2.54 mm to (124.5, 26.7)
- moved R8 2.54 mm to (152.4, 26.7)
- moved D1 1.27 mm to (137.2, 35.6)
Connections:
- D1 pad 1: Net-(D1-Pad1) -> ~HSync
- R10 pad 1: GND -> Net-(J1-Pad1)
- R10 pad 2: Net-(Q2-Pad1) -> Net-(R10-Pad2)
- R4 pad 1: Net-(D1-Pad2) -> VCC
- R4 pad 2: VCC -> Net-(D1-Pad2)
- R8 pad 1: Net-(J1-Pad1) -> Net-(R10-Pad2)
- R8 pad 2: Net-(Q2-Pad1) -> Net-(D1-Pad2)
- R9 pad 1: GND -> VCC
- U12 pad 10: GND -> VCC
- U12 pad 12: GND -> VCC
- U12 pad 13: GND -> VCC
- U12 pad 4: GND -> VCC
- U12 pad 5: GND -> VCC
- U12 pad 7: GND -> VCC
- U15 pad 15: ~RowClk -> RowClk
- U16 pad 13: GND -> VCC
- U16 pad 6: VCC -> GND
- U18 pad 2: VCC -> Net-(R11-Pad1)
- U18 pad 39: CPU_PHI2 -> Net-(U18-Pad39)
- U19 pad 12: Net-(U19-Pad12) -> RowClk
- U19 pad 13: Net-(U19-Pad13) -> ~DelayedRowClk
- U19 pad 2: CPU_PHI2 -> CPU_PHI0
- U19 pad 5: CPU_PHI2 -> CPU_PHI0
- U2 pad 10: ~VSync -> (no net)
- U2 pad 12: ~RowClk -> Net-(U19-Pad11)
- U2 pad 5: 2MHz -> ~2MHz
- U2 pad 8: Net-(D1-Pad1) -> (no net)
- U2 pad 9: ~HSync -> (no net)
- U6 pad 1: Net-(U6-Pad1) -> VCC
- U6 pad 12: ~RowClk -> RowClk
- U6 pad 8: Net-(U6-Pad8) -> ~DelayedRowClk
- U6 pad 9: Net-(U6-Pad1) -> Net-(U6-Pad9)
Routing:
- net 8MHz: track 63.5 -> 320.7 mm, vias 4 -> 8
- net A15: track 40.6 -> 251.9 mm, vias 1 -> 4
- net VSync: track 20.3 -> 202.8 mm, vias 0 -> 2
- net ~DelayedRowClk: track 0.00 -> 176.9 mm, vias 0 -> 2
- net ~RowClk: track 327.1 -> 164.7 mm, vias 8 -> 4
- net A14: track 38.1 -> 200.0 mm, vias 2 -> 4
- net A12: track 38.1 -> 183.4 mm, vias 2 -> 4
- net /Memory Controller/~CPUBUS: track 94.0 -> 227.4 mm, vias 6 -> 7
- net A13: track 40.6 -> 168.4 mm, vias 2 -> 5
- net ~ROMCS: track 30.5 -> 155.9 mm, vias 1 -> 2
- net CPU_PHI0: track 20.3 -> 144.6 mm, vias 1 -> 2
- net Net-(D1-Pad1): track 115.4 -> 0.00 mm, vias 2 -> 0
- net CPU_PHI2: track 39.2 -> 152.2 mm, vias 3 -> 4
- net HOn: track 62.3 -> 170.0 mm, vias 2 -> 4
- net RowClk: track 218.0 -> 323.8 mm, vias 8 -> 12
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Other:
- copper layers 2 -> 4
